Commit message: edit urdf file

File: src/bgr_description/urdf/bgr.urdf.xacro (robot description, xacro)
@@ -118,5 +118,4 @@
     <limit lower="-0.6" upper="0.6" effort="100" velocity="100" />
     <dynamics damping="0.1" friction="0.1" />
-    <mimic joint="Steering_fr_joint" multiplier="-1" offset="0" />
   </joint>
   <link name="Wheel_fl">
